File: KiCad/Leaf_BME680.kicad_pcb (KiCad board)
At the start: 4 copper layers, 20 x 20 mm, 8 parts, among them CN1 LeafIF, U1 BME680

Commit message: update pcb
Parts:
- added R5: 0R, Resistor_SMD:R_0603_1608Metric, F.Cu at (40.0, 31.7)
- added R6: 0R, Resistor_SMD:R_0603_1608Metric, F.Cu at (38.4, 31.7)
- CN1: footprint Leafony:CN_F29_B29 -> Trillion-Node:CN_F29_B29
- moved R4 2.77 mm to (32.3, 32.2)
- moved R2 1.58 mm to (39.9, 38.3)
- moved R1 1.48 mm to (39.9, 41.7)
- moved R3 1.08 mm to (32.3, 34.0)
- moved C1 0.66 mm to (31.7, 37.9)
- moved U1 0.58 mm to (35.0, 37.9)
- moved C2 0.24 mm to (35.0, 41.3)
- moved CN1 0.07 mm to (29.0, 28.5)
Connections:
- R3 pad 2: /SCK -> Net-(R3-Pad2)
- R4 pad 2: /SDA -> Net-(R4-Pad2)
- U1 pad 3: /SDA -> Net-(R3-Pad2)
- U1 pad 4: /SCK -> Net-(R4-Pad2)
Routing:
- net /SCK: track 16.4 -> 2.05 mm, vias 3 -> 1
- net Net-(R4-Pad2): track 0.00 -> 13.8 mm, vias 0 -> 2
- net /SDA: track 12.9 -> 2.35 mm
- net Net-(R3-Pad2): track 0.00 -> 10.2 mm
- net +3V3: track 13.0 -> 15.0 mm, vias 8 -> 7
- net GND: track 10.1 -> 11.7 mm, vias 10 -> 7
- net Net-(R1-Pad2): track 4.75 -> 5.52 mm
Other:
- net class Default: via_dia 0.5 -> 0.6
- rule pad_to_mask_clearance: 0.1 -> 0.2
- rule via_min_size: 0.5 -> 0.6
