File: KiCad/Leaf_BME680.sch (KiCad schematic (older format))
At the start: 8 parts, among them CN1 LeafIF, U1 BME680

Commit message: update pcb
Parts:
- added R5, R6: 0R, Resistor_SMD:R_0603_1608Metric, symbol Device:R
Connections:
- net SCK: now also R5.2; no longer R3.2, U1.4 (SCK)
- net SDA: now also R6.2; no longer R4.2, U1.3 (SDI)
- new net: R3.2, R6.1, U1.3 (SDI)
- new net: R4.2, R5.1, U1.4 (SCK)
Other:
- note added: "CSB\nI2C address bit 0\nGND: '0'; VDD: '1';"
- note removed: "SDO\nI2C address bit 0\nGND:0; VDD:1"
- moved on the sheet: CN1
